Commit message: 清理: 移动 mini.world 到 gazebo_worlds, 删除无用 maps/models
- mini.world: src/ackermann_robot/worlds/ → src/gazebo_worlds/worlds/
- 删除 ackermann_robot/models/ (空占位)
- 删除 ackermann_robot/worlds/ (除 mini.world 外的空 world)
- 删除 gazebo_worlds 中大量未使用的世界/地图文件
- map.launch.py: world 路径改为引用 gazebo_worlds
- ackermann_robot/CMakeLists.txt: 移除 worlds/models 安装
- gazebo_worlds: 新增 CMakeLists.txt + package.xml
- sensors.xacro: 小修改

File: src/ackermann_robot/xacro/sensors.xacro (robot description, xacro)
@@ -23,5 +23,5 @@
         <child link="laser_link" />
     </joint>
-    <!-- 单线360°激光雷达（原3D Velodyne已更换） -->
+    <!-- 单线360°激光雷达 -->
     <gazebo reference="laser_link">
         <material>Gazebo/Grey</material>
@@ -159,38 +159,3 @@
         </sensor>
     </gazebo>
-    <!-- <link name="rtk_link">
-        <inertial>
-            <mass value="0.6548" />
-            <inertia ixx="0.00081" ixy="-9.5e-11" ixz="1.19e-06" iyy="0.00081" iyz="-8.5e-11" izz="0.00139" />
-        </inertial>
-        <visual>
-            <geometry> <mesh filename="package://ackermann_robot/meshes/top_akm_bs_robot_meshes/rtk_link.STL" /> </geometry>
-            <material name="white"/>
-        </visual>
-        <collision>
-             <geometry> <mesh filename="package://ackermann_robot/meshes/top_akm_bs_robot_meshes/rtk_link.STL" /> </geometry>
-        </collision>
-    </link>
-    <joint name="rtk_joint" type="fixed">
-        <origin xyz="-0.043328 0.00081 0.20739" rpy="0 0 0" />
-        <parent link="base_link" />
-        <child link="rtk_link" />
-    </joint>
-    <gazebo reference="rtk_link">
-        <material>Gazebo/Blue</material>
-        <sensor name="rtk_gps" type="gps">
-            <always_on>true</always_on>
-            <update_rate>50.0</update_rate>
-            <gps>
-                <position_sensing>
-                    <horizontal> <noise type="gaussian"> <mean>0.0</mean> <stddev>0.01</stddev> </noise> </horizontal>
-                    <vertical> <noise type="gaussian"> <mean>0.0</mean> <stddev>0.01</stddev> </noise> </vertical>
-                </position_sensing>
-            </gps>
-            <plugin name="gps_controller" filename="libgazebo_ros_gps_sensor.so">
-                <ros> <remapping>~/out:=/gps/fix</remapping> </ros>
-                <frame_name>rtk_link</frame_name>
-            </plugin>
-        </sensor>
-    </gazebo> -->
 </robot>
